Commit message: [Add] square & coffee scene

File: fr3_husky_description/mjcf/dual_fr3_husky_coffee.xml.xacro (robot description, xacro)
@@ -20,5 +20,5 @@
     <xacro:include filename="$(find fr3_husky_description)/mjcf/realsense_d435i.xml.xacro"/>
     <xacro:include filename="$(find fr3_husky_description)/mjcf/azure_kinect.xml.xacro"/>
-    <xacro:include filename="$(find fr3_husky_description)/mjcf/threading_scene.xml.xacro"/>
+    <xacro:include filename="$(find fr3_husky_description)/mjcf/coffee_scene.xml.xacro"/>
     <xacro:include filename="$(find fr3_husky_description)/mjcf/assets/d435i_assets.xml.xacro" />
     <xacro:include filename="$(find fr3_husky_description)/mjcf/assets/azure_kinect_assets.xml.xacro" />
@@ -148,5 +148,10 @@
         <material name="floorplane" reflectance="0.01" shininess="0.0" specular="0.0" texrepeat="2 2" texture="texplane" texuniform="true"/>
         <texture file="$(find fr3_husky_description)/textures/ceramic.png" type="cube" name="tex-ceramic"/>
+        <material name="ceramic" reflectance="0.5" texrepeat="1 1" texture="tex-ceramic" texuniform="true"/>
         <material name="table_ceramic" reflectance="0.0" shininess="0.0" specular="0.2" texrepeat="1 1" texture="tex-ceramic"/>
+        <texture file="$(find fr3_husky_description)/textures/steel-scratched.png" type="cube" name="steel-metal"/>
+        <texture file="$(find fr3_husky_description)/textures/brass-ambra.png" type="cube" name="brass-metal"/>
+        <material name="smetal" reflectance="1.0" shininess="1.0" specular="1.0" texrepeat="1 1" texture="steel-metal" texuniform="true"/>
+        <material name="bmetal" reflectance="1.0" shininess="1.0" specular="1.0" texrepeat="1 1" texture="brass-metal" texuniform="true"/>
         <texture file="$(find fr3_husky_description)/textures/steel-brushed.png" type="cube" name="tex-steel-brushed"/>
         <material name="table_legs_metal" reflectance="0.8" shininess="0.8" texrepeat="1 1" texture="tex-steel-brushed"/>
@@ -157,4 +162,8 @@
         <material name="ring_gray" rgba="0.85 0.85 0.85 1" />
         <mesh name="bowl_mesh" file="$(find fr3_husky_description)/meshes/cup_nohandle.stl" scale="1.2 1.2 0.05" />
+        <mesh name="coffee_body_mesh" file="$(find fr3_husky_description)/meshes/coffee_body.stl" scale="0.01 0.01 0.01"/>
+        <mesh name="coffee_lid_mesh" file="$(find fr3_husky_description)/meshes/coffee_lid.stl" scale="0.01 0.01 0.01"/>
+        <mesh name="coffee_base_mesh" file="$(find fr3_husky_description)/meshes/coffee_base.stl" scale="0.01 0.01 0.01"/>
+        <mesh name="coffee_pod_mesh" file="$(find fr3_husky_description)/meshes/coffee_pod.stl" scale="0.018 0.018 0.018"/>
         <xacro:fr3_assets arm_id="$(arg arm_id)"/>
         <xacro:franka_hand_assets/>
@@ -178,5 +187,5 @@
                 fovy="55"
                 resolution="640 480" />
-        <xacro:threading_scene/>
+        <xacro:coffee_scene/>
         <body name="root" pos="0 0 0">
             <joint name="world_joint" type="free" stiffness="0" damping="0" frictionloss="0" armature="0" />

File: fr3_husky_description/mjcf/dual_fr3_husky_square.xml.xacro (robot description, xacro)
@@ -20,5 +20,5 @@
     <xacro:include filename="$(find fr3_husky_description)/mjcf/realsense_d435i.xml.xacro"/>
     <xacro:include filename="$(find fr3_husky_description)/mjcf/azure_kinect.xml.xacro"/>
-    <xacro:include filename="$(find fr3_husky_description)/mjcf/threading_scene.xml.xacro"/>
+    <xacro:include filename="$(find fr3_husky_description)/mjcf/square_scene.xml.xacro"/>
     <xacro:include filename="$(find fr3_husky_description)/mjcf/assets/d435i_assets.xml.xacro" />
     <xacro:include filename="$(find fr3_husky_description)/mjcf/assets/azure_kinect_assets.xml.xacro" />
@@ -149,4 +149,8 @@
         <texture file="$(find fr3_husky_description)/textures/ceramic.png" type="cube" name="tex-ceramic"/>
         <material name="table_ceramic" reflectance="0.0" shininess="0.0" specular="0.2" texrepeat="1 1" texture="tex-ceramic"/>
+        <texture file="$(find fr3_husky_description)/textures/steel-scratched.png" type="cube" name="steel-metal"/>
+        <texture file="$(find fr3_husky_description)/textures/brass-ambra.png" type="cube" name="brass-metal"/>
+        <material name="smetal" reflectance="1.0" shininess="1.0" specular="1.0" texrepeat="1 1" texture="steel-metal" texuniform="true"/>
+        <material name="bmetal" reflectance="1.0" shininess="1.0" specular="1.0" texrepeat="1 1" texture="brass-metal" texuniform="true"/>
         <texture file="$(find fr3_husky_description)/textures/steel-brushed.png" type="cube" name="tex-steel-brushed"/>
         <material name="table_legs_metal" reflectance="0.8" shininess="0.8" texrepeat="1 1" texture="tex-steel-brushed"/>
@@ -178,5 +182,5 @@
                 fovy="55"
                 resolution="640 480" />
-        <xacro:threading_scene/>
+        <xacro:square_scene/>
         <body name="root" pos="0 0 0">
             <joint name="world_joint" type="free" stiffness="0" damping="0" frictionloss="0" armature="0" />

File: fr3_husky_description/mjcf/dual_fr3_husky_threepieceassembly.xml.xacro (robot description, xacro)
@@ -149,4 +149,8 @@
         <texture file="$(find fr3_husky_description)/textures/ceramic.png" type="cube" name="tex-ceramic"/>
         <material name="table_ceramic" reflectance="0.0" shininess="0.0" specular="0.2" texrepeat="1 1" texture="tex-ceramic"/>
+        <texture file="$(find fr3_husky_description)/textures/steel-brushed.png" type="cube" name="tex-steel-brushed"/>
+        <material name="table_legs_metal" reflectance="0.8" shininess="0.8" texrepeat="1 1" texture="tex-steel-brushed"/>
+        <texture file="$(find fr3_husky_description)/textures/light-gray-plaster.png" type="2d" name="tex-light-gray-plaster"/>
+        <material name="walls_mat" reflectance="0.0" shininess="0.1" specular="0.1" texrepeat="3 3" texture="tex-light-gray-plaster" texuniform="true"/>
         <material name="env_red" rgba="1 0.072272 0.039546 1" />
         <material name="env_blue" rgba="0.024157 0.445201 0.737911 1" />
@@ -206,4 +210,10 @@
         </body>
     </worldbody>
+    <equality>
+        <weld name="weld_right_tcp" body1="right_fr3_hand_tcp" body2="obj"
+              active="false" solref="0.02 1" solimp="0.9 0.95 0.001"/>
+        <weld name="weld_left_tcp" body1="left_fr3_hand_tcp" body2="obj"
+              active="false" solref="0.02 1" solimp="0.9 0.95 0.001"/>
+    </equality>
     <!-- Wheel actuators -->
     <xacro:husky_wheel_actuator prefix="" as_two_wheels="false"/>

File: fr3_husky_description/mjcf/threading_scene.xml.xacro (robot description, xacro)
@@ -2,4 +2,7 @@
 <mujoco xmlns:xacro="http://www.ros.org/wiki/xacro">
     <xacro:macro name="threading_scene">
+        <!-- <geom pos="-1.2 0 1.5" quat="0.5 0.5 0.5 0.5"
+              size="1.5 1.5 0.01" type="box" conaffinity="0" contype="0"
+              group="1" name="wall_rear_visual" material="walls_mat"/> -->
         <body name="goal_marker" pos="0 0 0">
             <joint name="goal_marker_joint" type="free"/>
@@ -18,7 +21,7 @@
                   friction="1 0.005 0.0001"/>
         </body>
-        <body name="needle_obj" pos="0.72 -0.2 1.0" quat="0.8660254 0 0 -0.5">
-            <freejoint name="needle_obj_joint"/>
-            <geom name="needle_obj_needle"
+        <body name="obj" pos="0.65 -0.4 0.8" quat="0 0 1 0">
+            <freejoint name="obj_joint"/>
+            <geom name="obj_needle"
                   type="box"
                   pos="0 -0.08 0"
@@ -29,5 +32,5 @@
                   solref="0.02 1"
                   solimp="0.9 0.95 0.001"/>
-            <geom name="needle_obj_handle"
+            <geom name="obj_handle"
                   type="box"
                   pos="0 0 0"
@@ -38,5 +41,5 @@
                   solimp="0.9 0.95 0.001"/>
         </body>
-        <body name="tripod_obj" pos="0.88 -0.40 0.8" quat="0.7071068 0 0 0.7071068"> # table 기준 차이 = (+0.08, -0.15, +0.1)
+        <body name="tripod_obj" pos="0.80 -0.40 0.8" quat="0.7071068 0 0 0.7071068">
             <geom name="tripod_obj_ring_0" type="box" pos="0 -0.01 0.078" size="0.005 0.002 0.002" rgba="0.7 0.56 0.36 1" density="100" friction="0.3 0.005 0.0001" solref="0.02 1" solimp="0.9 0.95 0.001"/>
             <geom name="tripod_obj_ring_1" type="box" pos="0 -0.006 0.078" size="0.005 0.002 0.002" rgba="0.7 0.56 0.36 1" density="100" friction="0.3 0.005 0.0001" solref="0.02 1" solimp="0.9 0.95 0.001"/>

File: fr3_husky_description/mjcf/threepieceassembly_scene.xml.xacro (robot description, xacro)
@@ -14,4 +14,7 @@
     </xacro:macro>
     <xacro:macro name="threepieceassembly_scene">
+        <!-- <geom pos="-1.2 0 1.5" quat="0.5 0.5 0.5 0.5"
+              size="1.5 1.5 0.01" type="box" conaffinity="0" contype="0"
+              group="1" name="wall_rear_visual" material="walls_mat"/> -->
         <!-- MimicGen ThreePieceAssembly object set:
              - table: TableArena-style tabletop with full size (0.8, 0.8, 0.05) and offset z=0.8
@@ -20,5 +23,5 @@
              - piece_2: 4-layer bridge piece, unit half-size 0.02
              Placement here is deterministic and chosen to sit on the FR3 Husky top plate. -->
-        <body name="threepieceassembly_table" pos="0.9 -0.25 0.7">
+        <body name="threepieceassembly_table" pos="0.9 -0.25 0.6">
             <geom name="threepieceassembly_table_top"
                   type="box"
@@ -30,5 +33,5 @@
                   solimp="0.9 0.95 0.001"/>
         </body>
-        <body name="base" pos="0.8 -0.25 0.880">
+        <body name="base" pos="0.8 -0.25 0.780">
             <freejoint name="base_joint"/>
             <xacro:threepieceassembly_voxel name="base_0_0_0" pos="-0.076 -0.076 0.0" size="0.019 0.019 0.019" density="10000" rgba="0.70 0.18 0.16 1"/>
@@ -49,5 +52,5 @@
             <xacro:threepieceassembly_voxel name="base_0_4_4" pos="0.076 0.076 0.0" size="0.019 0.019 0.019" density="10000" rgba="0.70 0.18 0.16 1"/>
         </body>
-        <body name="piece_1" pos="0.78 0.0 1.012" euler="0 0 1.5708">
+        <body name="piece_1" pos="0.8 -0.25 0.912" euler="0 0 1.5708">
             <freejoint name="piece_1_joint"/>
             <xacro:threepieceassembly_voxel name="piece_1_0_0_0" pos="-0.034 -0.034 -0.034" size="0.017 0.017 0.017" density="100" rgba="0.78 0.25 0.22 1"/>
@@ -67,6 +70,6 @@
             <xacro:threepieceassembly_voxel name="piece_1_2_1_2" pos="0.0 0.034 0.034" size="0.017 0.017 0.017" density="100" rgba="0.78 0.25 0.22 1"/>
         </body>
-        <body name="piece_2" pos="0.9 -0.45 0.941" euler="0 0 1.5708">
-            <freejoint name="piece_2_joint"/>
+        <body name="obj" pos="0.8 -0.4 0.841" euler="0 0 1.5708">
+            <freejoint name="obj_joint"/>
             <xacro:threepieceassembly_voxel name="piece_2_0_0_0" pos="-0.04 -0.04 -0.06" size="0.02 0.02 0.02" density="100" rgba="0.86 0.38 0.28 1"/>
             <xacro:threepieceassembly_voxel name="piece_2_0_0_1" pos="-0.04 0.0 -0.06" size="0.02 0.02 0.02" density="100" rgba="0.86 0.38 0.28 1"/>
